File: Electronics/PowerRails.kicad_sch (KiCad schematic)
At the start: 17 parts, among them U3 LM2596S-ADJ, U4 AMS1117-3.3 (Potentially swap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

Commit message: Electronics release 1.0
Parts:
- removed TP9: 12V, TestPoint:TestPoint_Pad_D1.0mm, symbol Connector:TestPoint
- added TP12: +12V, TestPoint:TestPoint_Pad_D1.0mm, symbol Connector:TestPoint
Connections:
- net +12V_{MOTOR}: now also TP12.1
- net +5V_{LREG}: no longer D4.1 (K), RV1.2
- net at L1.1, U3.2 (OUT): now also D4.1 (K)
Other:
- moved on the sheet: D4, L1, R12, RV1
