File: Electronics/ShutterRetroFit.kicad_pcb (KiCad board)
At the start: 4 copper layers, 50 x 50 mm, 86 parts, among them IC1 NCP5104DR2G, IC2 NCP5104DR2G, J1 AMPHENOL_12402012E212A, J2 AS5600, J3 PWR_IN+, J4 EXP, J5 CONTROL, J6 PWR_IN-, J7 Motor A, J8 Motor B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

Commit message: Electronics release 1.0
Parts:
- removed C7, C8: 0.1uF, Capacitor_SMD:C_0603_1608Metric_Pad1.08x0.95mm_HandSolder
- removed H4: MountingHole_Pad, MountingHole:MountingHole_3.2mm_M3_DIN965_Pad
- removed J4: EXP, Connector_PinHeader_2.54mm:PinHeader_1x06_P2.54mm_Vertical
- removed R15, R17, R3, R4: 1k, Resistor_SMD:R_0603_1608Metric_Pad0.98x0.95mm_HandSolder
- removed R16: W_{shunt}, CustomLibrary:Shunt Wire
- removed R18: 20k, Resistor_SMD:R_0603_1608Metric_Pad0.98x0.95mm_HandSolder
- removed TP13: V-, TestPoint:TestPoint_Pad_D1.0mm
- removed TP14: V+, TestPoint:TestPoint_Pad_D1.0mm
- removed TP9: 12V, TestPoint:TestPoint_Pad_D1.0mm
- added C21: 0.1uF, Capacitor_SMD:C_0603_1608Metric_Pad1.08x0.95mm_HandSolder, F.Cu at (145.0, 103.0)
- added D1: RB751ASA-40FHT2RB, CustomLibrary:D_SOD-882_Handsoldered, F.Cu at (125.1, 123.6)
- added D2: RB751ASA-40FHT2RB, CustomLibrary:D_SOD-882_Handsoldered, F.Cu at (147.4, 123.6)
- added IC3: INA2180A2QDGKRQ1, CustomLibrary:SOP65P490X110-8N, F.Cu at (140.7, 103.0)
- added R26: MFSA1206R0100FCM, Resistor_SMD:R_1206_3216Metric_Pad1.30x1.75mm_HandSolder, F.Cu at (140.4, 107.1)
- added TP15: V-, TestPoint:TestPoint_Pad_D1.0mm, F.Cu at (136.2, 104.5)
- added TP16: V+, TestPoint:TestPoint_Pad_D1.0mm, F.Cu at (135.9, 102.3)
- J2: value AS5600 -> ACCESSORY
- L1: value 470 -> 47uH
- R13: value 20k -> 0
- R14: value CSM2512R1F1L00S9 -> 0; footprint Resistor_SMD:R_2512_6332Metric_Pad1.40x3.35mm_HandSolder -> Resistor_SMD:R_0603_1608Metric_Pad0.98x0.95mm_HandSolder
- R24, R25: value 0 -> 1k
- TP12: value M_{SENSE} -> +12V
- moved U3 176.1 mm to (96.8, 108.3), turned to 180 degrees
- moved L1 170.6 mm to (98.0, 95.6)
- moved TP10 166.1 mm to (112.3, 93.0)
- moved C9 162.3 mm to (98.7, 118.5), turned to 180 degrees
- moved RV1 160.9 mm to (107.8, 98.2), turned to -90 degrees
- moved C10 159.5 mm to (105.3, 115.0)
- moved C11 157.3 mm to (101.2, 86.3), turned to -90 degrees
- moved F1 157.2 mm to (109.2, 129.3), turned to 90 degrees
- moved C12 154.8 mm to (95.6, 82.9), turned to 180 degrees
- moved TP11 153.1 mm to (122.3, 75.8)
- moved R12 151.5 mm to (108.2, 107.5), turned to -90 degrees
- moved TP5 145.6 mm to (123.9, 115.8), turned to 180 degrees
- moved D4 140.1 mm to (111.7, 105.4), turned to 90 degrees
- moved R10 137.5 mm to (123.6, 112.6), turned to -90 degrees
- moved R24 137.4 mm to (128.6, 125.3), turned to 180 degrees
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Connections:
- C4 pad 1: /MCU_{VIN} -> /+3v3
- D4 pad 1: +5V_{LREG} -> Net-(D4-K)
- F2 pad 2: /+3v3_{EXP} -> /+3v3
- J2 pad 2: GND -> /IO33
- J2 pad 4: /AS5600_{SDA} -> /SENS_{SCL}
- J2 pad 5: /AS5600_{SCL} -> /SENS_{SDA}
- J2 pad 6: /+3v3_{EXP} -> +5V_{LREG}
- J3 pad 2: (no net) -> +12V
- J5 pad 2: /BTN_{DOWN} -> /BTN_{UP}
- J5 pad 3: /BTN_{UP} -> /BTN_{DOWN}
- J6 pad 2: (no net) -> GND
- J7 pad 2: (no net) -> /Motor/L_{MID}
- J8 pad 2: (no net) -> /Motor/R_{MID}
- L1 pad 1: Net-(U3-OUT) -> Net-(D4-K)
- R13 pad 1: /M_{SENSE} -> Net-(IC2-BRIDGE)
- R13 pad 2: Net-(U5--) -> /Motor/L_{MID}
- R14 pad 1: +12v_{EXP} -> Net-(IC1-BRIDGE)
- R14 pad 2: Net-(R14-Pad2) -> /Motor/R_{MID}
- RV1 pad 2: +5V_{LREG} -> unconnected-(RV1-Pad2)
- TP12 pad 1: /M_{SENSE} -> +12V_{MOTOR}
- U2 pad 10: /EXP_{02} -> unconnected-(U2-IO25-Pad10)
- U2 pad 11: /EXP_{01} -> /H_{DRIVER_RIGHT_CONTROL}
- U2 pad 14: /H_{DRIVER_LEFT_CONTROL} -> unconnected-(U2-IO12-Pad14)
- U2 pad 2: /MCU_{VIN} -> /+3v3
- U2 pad 23: /H_{DRIVER_RIGHT_CONTROL} -> unconnected-(U2-IO15-Pad23)
- U2 pad 27: /M_{SENSE} -> unconnected-(U2-IO16-Pad27)
- U2 pad 28: /D_{POWER} -> unconnected-(U2-IO17-Pad28)
- U2 pad 33: /AS5600_{SDA} -> /SENS_{SDA}
- U2 pad 36: /AS5600_{SCL} -> /SENS_{SCL}
- U2 pad 37: unconnected-(U2-IO23-Pad37) -> /D_{POWER}
- U2 pad 6: unconnected-(U2-IO34-Pad6) -> /M_{SENSE}
- U2 pad 9: unconnected-(U2-IO33-Pad9) -> /IO33
- U3 pad 2: Net-(U3-OUT) -> Net-(D4-K)
Routing:
- net +5V_{LREG}: track 0.00 -> 106.8 mm
- net GND: track 0.00 -> 81.8 mm, vias 0 -> 42
- net /Motor/L_{MID}: track 0.00 -> 71.6 mm, vias 0 -> 2
- net /BTN_{DOWN}: track 0.00 -> 64.5 mm, vias 0 -> 2
- net /D_{ERROR}: track 0.00 -> 62.7 mm, vias 0 -> 2
- net /D_{POWER}: track 0.00 -> 61.7 mm, vias 0 -> 2
- net /BTN_{UP}: track 0.00 -> 61.5 mm, vias 0 -> 2
- net /IO33: track 0.00 -> 59.6 mm, vias 0 -> 2
- net /Motor/R_{MID}: track 0.00 -> 57.8 mm, vias 0 -> 2
- net /D_{STATUS}: track 0.00 -> 57.5 mm, vias 0 -> 2
- net /H_{DRIVER_RIGHT_CONTROL}: track 0.00 -> 51.8 mm, vias 0 -> 2
- net /H_{DRIVER_RIGHT_EN}: track 0.00 -> 51.6 mm, vias 0 -> 4
- net /SENS_{SCL}: track 0.00 -> 47.2 mm, vias 0 -> 2
- net /H_{DRIVER_LEFT_EN}: track 0.00 -> 43.8 mm, vias 0 -> 2
- net /SENS_{SDA}: track 0.00 -> 40.1 mm, vias 0 -> 2
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- added copper zone on B.Cu, net +12v_{EXP}
- removed copper zone on B.Cu, net GND
- removed copper zone on In2.Cu, net GND
Other:
- board size 50 x 50 mm -> 90 x 68.3 mm
- copper layers 4 -> 2
- board text added: "ACCESSORY"
- board text added: "Explosions waiting to happen..."
- board text added: "FEEDBACK"
- board text added: "MOTOR A"
- board text added: "MOTOR B"
- board text added: "Motor Driver Rev 1.0"
- board text added: "Ripples ahead"
- board text added: "V+"
- board text added: "V-"
