File: Electronics/motor_sch.kicad_sch (KiCad schematic)
At the start: 40 parts, among them IC1 NCP5104DR2G, IC2 NCP5104DR2G, IC3 INA2180A2QDGKRQ1, J7 Motor A, J8 Motor B, M1 YG2738, Q5 SiSS52DN-T1-GE3, Q6 SiSS52DN-T1-GE3, Q7 SiSS52DN-T1-GE3, Q8 SiSS52DN-T1-GE3

Commit message: Electronics release 1.0
Parts:
- removed J7: Motor A, CustomLibrary:CONN_726386-2_TEC, symbol Connector:Conn_01x01_Pin
- removed J8: Motor B, CustomLibrary:CONN_726386-2_TEC, symbol Connector:Conn_01x01_Pin
- added J7: Motor A, symbol Connector:Conn_01x02_Pin
- added J8: Motor B, symbol Connector:Conn_01x02_Pin
- added R13, R14: 0, Resistor_SMD:R_0603_1608Metric_Pad0.98x0.95mm_HandSolder, symbol Device:R_Small
- IC1, IC2: footprint SOIC127P600X175-8N -> CustomLibrary:SOIC127P600X175-8N
- IC3: footprint SOP65P490X110-8N -> CustomLibrary:SOP65P490X110-8N
- Q5, Q6, Q7, Q8: footprint SISS94DNT1GE3 -> CustomLibrary:SISS94DNT1GE3
- R26: value CSM2512R1F1L00S9 -> MFSA1206R0100FCM; footprint Resistor_SMD:R_2512_6332Metric_Pad1.40x3.35mm_HandSolder -> Resistor_SMD:R_1206_3216Metric_Pad1.30x1.75mm_HandSolder
Connections:
- net L_{MID}: now also J7.1 (Pin_1), J7.2 (Pin_2), R13.2
- net R_{MID}: now also J8.1 (Pin_1), J8.2 (Pin_2), R14.2
- net at C16.1, C19.1, IC2.6 (BRIDGE): now also R13.1
- net at C17.1, C20.1, IC1.6 (BRIDGE): now also R14.1
Other:
- note added: "Only poulate one of these at any time Aiming at 10mV drop per amp, 50x Gain"
- note removed: "Only poulate one of these at any time Aiming at 1mV drop per amp, with a 100x gain."
